File: STMBlueLine.kicad_pcb (KiCad board)
At the start: 2 copper layers, 0 parts

Commit message: ADD : Footprint assignment. FIX : Various ERC rules.
Parts:
- added 1: M.2-B-KEY, M.2-Templates:M.2-B-KEY, F.Cu at (35.3, 65.5)
- added C1: 100nF, Capacitor_SMD:C_0402_1005Metric, F.Cu at (50.3, 39.7)
- added C10: 1uF, Capacitor_SMD:C_0402_1005Metric, F.Cu at (56.0, 41.7)
- added C11: 9pF, Capacitor_SMD:C_0402_1005Metric, F.Cu at (56.0, 43.6)
- added C12: 9pF, Capacitor_SMD:C_0402_1005Metric, F.Cu at (56.0, 45.6)
- added C13: 10uF, Capacitor_SMD:C_0402_1005Metric, F.Cu at (70.5, 63.5)
- added C14: 100nF, Capacitor_SMD:C_0402_1005Metric, F.Cu at (58.9, 39.7)
- added C15: 100nF, Capacitor_SMD:C_0402_1005Metric, F.Cu at (58.9, 41.7)
- added C16: 22uF, Capacitor_SMD:C_0402_1005Metric, F.Cu at (87.7, 21.2)
- added C17: 22uF, Capacitor_SMD:C_0402_1005Metric, F.Cu at (87.7, 23.2)
- added C18: 100nF, Capacitor_SMD:C_0402_1005Metric, F.Cu at (25.2, 69.2)
- added C19: 100nF, Capacitor_SMD:C_0402_1005Metric, F.Cu at (50.3, 70.0)
- added C2: 100nF, Capacitor_SMD:C_0402_1005Metric, F.Cu at (50.3, 41.7)
- added C20: 1uF, Capacitor_SMD:C_0402_1005Metric, F.Cu at (25.2, 71.2)
- added C21: 1uF, Capacitor_SMD:C_0402_1005Metric, F.Cu at (50.3, 71.9)
- added C22: 100nF, Capacitor_SMD:C_0402_1005Metric, F.Cu at (25.2, 73.1)
- added C23: 1uF, Capacitor_SMD:C_0402_1005Metric, F.Cu at (25.2, 75.1)
- added C24: 100nF, Capacitor_SMD:C_0402_1005Metric, F.Cu at (50.3, 73.9)
- added C25: 1uF, Capacitor_SMD:C_0402_1005Metric, F.Cu at (50.3, 75.9)
- added C26: 100nF, Capacitor_SMD:C_0402_1005Metric, F.Cu at (25.2, 77.1)
- added C27: 1uF, Capacitor_SMD:C_0402_1005Metric, F.Cu at (25.2, 79.0)
- added C28: 100nF, Capacitor_SMD:C_0402_1005Metric, F.Cu at (50.3, 77.8)
- added C29: 1uF, Capacitor_SMD:C_0402_1005Metric, F.Cu at (50.3, 79.8)
- added C3: 100nF, Capacitor_SMD:C_0402_1005Metric, F.Cu at (50.3, 43.6)
- added C30: 100nF, Capacitor_SMD:C_0402_1005Metric, F.Cu at (28.1, 69.2)
- added C31: 1uF, Capacitor_SMD:C_0402_1005Metric, F.Cu at (28.1, 71.2)
- added C32: 100nF, Capacitor_SMD:C_0402_1005Metric, F.Cu at (53.1, 70.0)
- added C33: 1uF, Capacitor_SMD:C_0402_1005Metric, F.Cu at (53.1, 71.9)
- added C34: 10uF, Capacitor_SMD:C_0402_1005Metric, F.Cu at (28.1, 73.1)
- added C35: 10uF, Capacitor_SMD:C_0402_1005Metric, F.Cu at (53.1, 73.9)
- added C36: 100nF, Capacitor_SMD:C_0402_1005Metric, F.Cu at (28.1, 75.1)
- added C37: 1uF, Capacitor_SMD:C_0402_1005Metric, F.Cu at (28.1, 77.1)
- added C38: 100nF, Capacitor_SMD:C_0402_1005Metric, F.Cu at (53.1, 75.9)
- added C39: 1uF, Capacitor_SMD:C_0402_1005Metric, F.Cu at (53.1, 77.8)
- added C4: 100nF, Capacitor_SMD:C_0402_1005Metric, F.Cu at (50.3, 45.6)
- added C40: 22uF, Capacitor_SMD:C_0402_1005Metric, F.Cu at (87.7, 25.1)
- added C41: 22uF, Capacitor_SMD:C_0402_1005Metric, F.Cu at (87.7, 27.1)
- added C42: 2.2uF, Capacitor_SMD:C_0402_1005Metric, F.Cu at (58.9, 43.6)
- added C43: 2.2uF, Capacitor_SMD:C_0402_1005Metric, F.Cu at (58.9, 45.6)
- added C5: 100nF, Capacitor_SMD:C_0402_1005Metric, F.Cu at (53.1, 39.7)
- added C6: 100nF, Capacitor_SMD:C_0402_1005Metric, F.Cu at (53.1, 41.7)
- added C7: 10uF, Capacitor_SMD:C_0402_1005Metric, F.Cu at (53.1, 43.6)
- added C8: 10nF, Capacitor_SMD:C_0402_1005Metric, F.Cu at (53.1, 45.6)
- added C9: 1uF, Capacitor_SMD:C_0402_1005Metric, F.Cu at (56.0, 39.7)
- added D1: LED, LED_SMD:LED_0402_1005Metric, F.Cu at (87.9, 29.1)
- added D2: D_TVS, Diode_SMD:D_0402_1005Metric, F.Cu at (73.7, 49.6)
- added D3: D_TVS, Diode_SMD:D_0402_1005Metric, F.Cu at (73.7, 51.6)
- added D4: D_TVS, Diode_SMD:D_0402_1005Metric, F.Cu at (73.7, 53.6)
- added D5: D_TVS, Diode_SMD:D_0402_1005Metric, F.Cu at (73.7, 55.5)
- added D6: D_TVS, Diode_SMD:D_0402_1005Metric, F.Cu at (73.7, 57.5)
- added D7: D_TVS, Diode_SMD:D_0402_1005Metric, F.Cu at (73.7, 59.5)
- added D8: D_TVS, Diode_SMD:D_0402_1005Metric, F.Cu at (73.7, 61.5)
- added FB1: 120R, Resistor_SMD:R_0402_1005Metric, F.Cu at (68.8, 34.6)
- added J1: Micro_SD_Card_Det1, random-footprints:TF15X15, F.Cu at (59.0, 57.8)
- added J2: USB_C_Receptacle_USB2.0_14P, Connector_USB:USB_C_Receptacle_G-Switch_GT-USB-7010ASV, F.Cu at (83.0, 54.0)
- added J3: Conn_01x04_Pin, Connector_PinHeader_2.54mm:PinHeader_1x04_P2.54mm_Vertical, F.Cu at (41.6, 70.5)
- added R1: 10k, Resistor_SMD:R_0402_1005Metric, F.Cu at (31.0, 76.5)
- added R10: 5.1k, Resistor_SMD:R_0402_1005Metric, F.Cu at (83.7, 59.7)
- added R11: 5.1k, Resistor_SMD:R_0402_1005Metric, F.Cu at (83.7, 61.6)
- added R12: 10k, Resistor_SMD:R_0402_1005Metric, F.Cu at (70.5, 61.5)
- added R13: 10k, Resistor_SMD:R_0402_1005Metric, F.Cu at (56.0, 77.3)
- added R14: 10k, Resistor_SMD:R_0402_1005Metric, F.Cu at (31.0, 78.5)
- added R15: 10k, Resistor_SMD:R_0402_1005Metric, F.Cu at (56.0, 79.3)
- added R2: 10k, Resistor_SMD:R_0402_1005Metric, F.Cu at (70.5, 49.6)
- added R3: 10k, Resistor_SMD:R_0402_1005Metric, F.Cu at (70.5, 51.6)
- added R4: 10k, Resistor_SMD:R_0402_1005Metric, F.Cu at (70.5, 53.6)
- added R5: 10k, Resistor_SMD:R_0402_1005Metric, F.Cu at (70.5, 55.5)
- added R6: 10k, Resistor_SMD:R_0402_1005Metric, F.Cu at (70.5, 57.5)
- added R7: 10k, Resistor_SMD:R_0402_1005Metric, F.Cu at (70.5, 59.5)
- added R8: 10k, Resistor_SMD:R_0402_1005Metric, F.Cu at (68.8, 36.5)
- added R9: 1.5k, Resistor_SMD:R_0402_1005Metric, F.Cu at (87.7, 31.1)
- added SW1: SW_Push, random-footprints:SW_TS-1088-AR02016, F.Cu at (70.8, 22.4)
- added SW2: SW_Push, random-footprints:SW_TS-1088-AR02016, F.Cu at (70.8, 26.9)
- added U1: STM32H750VBTx, Package_QFP:LQFP-100_14x14mm_P0.5mm, F.Cu at (58.1, 29.5)
- added U2: TLV320AIC3104IRHBR, random-footprints:QFN50P500X500X100-33N, F.Cu at (33.6, 71.9)
- added U3: TLV320AIC3104IRHBR, random-footprints:QFN50P500X500X100-33N, F.Cu at (58.7, 72.6)
- added U4: LD1117S33TR_SOT223, Package_TO_SOT_SMD:SOT-223-3_TabPin2, F.Cu at (81.3, 24.4)
- added U5: USBLC6-2SC6, Package_TO_SOT_SMD:SOT-23-6, F.Cu at (79.7, 61.1)
- added U6: LD1117S18TR_SOT223, Package_TO_SOT_SMD:SOT-223-3_TabPin2, F.Cu at (81.3, 32.7)
- added Y1: 16MHz, Crystal:Crystal_SMD_3225-4Pin_3.2x2.5mm, F.Cu at (70.0, 31.3)
Other:
- board outline added: 22 x 42 mm
